Commit message: Harvest Dell calibration wizard field fixes

File: so101_description/urdf/so101_arm.urdf.xacro (robot description, xacro)
@@ -5,4 +5,5 @@
   <xacro:arg name="add_transmissions" default="false"/>
   <xacro:arg name="use_ros2_control" default="false"/>
+  <xacro:arg name="control_variant" default="$(arg variant)"/> <!-- leader | follower; controls command interfaces -->
   <xacro:arg name="hardware_type" default="mock"/>
   <xacro:arg name="usb_port" default="/dev/ttyUSB0"/>
@@ -18,4 +19,5 @@
   <xacro:property name="use_ros2_control" value="$(arg use_ros2_control)"/>
   <xacro:property name="variant" value="$(arg variant)"/>
+  <xacro:property name="control_variant" value="$(arg control_variant)"/>
   <xacro:property name="enable_static_cam" value="$(arg enable_static_cam)"/>
   <xacro:property name="enable_wrist_cam" value="$(arg enable_wrist_cam)"/>
@@ -44,5 +46,5 @@
   <xacro:if value="${use_ros2_control}">
     <xacro:so101_ros2_control
-      variant="${variant}"
+      variant="${control_variant}"
       hardware_type="$(arg hardware_type)"
       usb_port="$(arg usb_port)"
